Commit message: update urdf (multiscan, imu, gps)

File: sick_wagen/urdf/sick_wagen.urdf (robot description, URDF)
Before this commit: robot whill_simulator, 16 links, 15 joints
Links:
- removed link sensor_arm_link
Joints:
- removed joint sensor_arm_joint
- joint gps_joint: origin xyz=0.12 0.25 1.03 rpy=0 0 0 -> xyz=-0.1 0.25 1.03 rpy=0 0 0
- joint imu_joint: origin xyz=-0.14 0 1.05 rpy=0 0 0 -> xyz=0.45 0 0.25 rpy=0 0 0
- joint multiscan_joint: origin xyz=-0.10 0 1.545 rpy=0 0 0 -> xyz=-0.10 0 1.03 rpy=0 0 0

Commit message: update urdf

File: sick_wagen/urdf/sick_wagen.urdf (robot description, URDF)
Before this commit: robot whill_simulator, 15 links, 14 joints
Joints:
- joint gps_joint: origin xyz=-0.1 0.25 1.03 rpy=0 0 0 -> xyz=-0.1 0.25 1.0 rpy=0 0 0
- joint multiscan_joint: origin xyz=-0.10 0 1.03 rpy=0 0 0 -> xyz=-0.10 0 0.92 rpy=0 0 0

Commit message: add rviz, modify rviz-multiscan

File: sick_wagen/urdf/sick_wagen.urdf (robot description, URDF)
Before this commit: robot whill_simulator, 15 links, 14 joints
Joints:
- joint multiscan_joint: origin xyz=-0.10 0 0.92 rpy=0 0 0 -> xyz=-0.10 0 0.92 rpy=3.141592 0 0

Commit message: feat: update localization parameters and add new point cloud data file - Change map_path to the correct file location - Enable odometry usage and set initial pose quaternion - Comment out robot state publisher node in launch file - Adjust IMU joint orientation in URDF

File: sick_wagen/urdf/sick_wagen.urdf (robot description, URDF)
Before this commit: robot whill_simulator, 15 links, 14 joints
Joints:
- joint imu_joint: origin xyz=0.45 0 0.25 rpy=0 0 0 -> xyz=0.45 0 0.25 rpy=0 0 -1.57
